File: Kikad_PCBs/PWM_JOSE_v1/PWM_JOSE_v1.sch (KiCad schematic (older format))
At the start: 32 parts, among them J1 Isense, J2 Out, J3 AlimOut, J4 AlimIn, Q1 BC548, Q2 BC558, U1 UC2844N, U2 PC817, U3 TL431

Commit message: PCB del pwm terminado
Parts:
- removed J1: Isense, symbol Conn_01x01
- removed J2: Out, symbol Conn_01x01
- added J1: signals, Connectors:bornier2, symbol Conn_01x02
- added Q3: Q_NPN_CBE, TO_SOT_Packages_THT:TO-92_Inline_Narrow_Oval, symbol Q_NPN_CBE
- added R15: RZ, Resistors_THT:R_Axial_DIN0414_L11.9mm_D4.5mm_P15.24mm_Horizontal, symbol R
- C1, C2, C3, C4, C5, C6, C7: footprint (none) -> Capacitors_THT:C_Disc_D5.0mm_W2.5mm_P2.50mm
- C8: footprint Capacitors_THT:CP_Axial_L10.0mm_D4.5mm_P15.00mm_Horizontal -> Capacitors_THT:C_Disc_D5.0mm_W2.5mm_P2.50mm
- D1: footprint (none) -> Diodes_THT:D_A-405_P7.62mm_Horizontal
- J3, J4: footprint (none) -> Connectors:bornier2
- Q1, Q2: footprint TO_SOT_Packages_THT:TO-92_Molded_Narrow -> TO_SOT_Packages_THT:TO-92_Inline_Narrow_Oval
- R1, R10, R11, R12, R13, R14, R2, R3, R4, R5, R6, R7, R8, R9: footprint (none) -> Resistors_THT:R_Axial_DIN0207_L6.3mm_D2.5mm_P7.62mm_Horizontal
- U1: footprint (none) -> Housings_DIP:DIP-8_W7.62mm_LongPads
- U3: footprint (none) -> TO_SOT_Packages_THT:TO-92_Inline_Wide
Connections:
- net +VDC: now also J3.2 (Pin_2), Q3.1 (C), R15.1; no longer J3.1 (Pin_1), R10.1, R11.1, R13.1
- net GNDS: now also J3.1 (Pin_1); no longer J3.2 (Pin_2)
- net at R11.2, R12.2, U2.2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: no longer D1.1 (K)
- net at R5.1: now also J1.2 (Pin_2)
- net at R6.1, R7.1: now also J1.1 (Pin_1)
- new net: Q3.3 (E), R10.1, R11.1, R13.1
- new net: D1.1 (K), Q3.2 (B), R15.2
Other:
- moved on the sheet: D1
