File: Kikad_PCBs/PWM_JOSE_v1/PWM_JOSE_v1.sch (KiCad schematic (older format))
At the start: 31 parts, among them J1 signals, J3 AlimOut, J4 AlimIn, Q1 BC548, Q2 BC558, U1 UC2844N, U2 PC817, U3 TL431

Commit message: pcb con esquematico y valores
Parts:
- Rbleeder: value 10k -> 100k
Changed lines of the file:
@@
 P 4550 2600
 F 0 "Rbleeder" V 4630 2600 50  0000 C CNN
-F 1 "10k" V 4550 2600 50  0000 C CNN
+F 1 "100k" V 4550 2600 50  0000 C CNN
 F 2 "Resistors_THT:R_Axial_DIN0207_L6.3mm_D2.5mm_P7.62mm_Horizontal" V 4480 2600 50  0001 C CNN
 F 3 "" H 4550 2600 50  0001 C CNN

Commit message: Placa final diseño completo.
Diseño kicad de la placa funcionando, falta hacer las modificaciones para que quede listo como para mandar a hacer, tambien modificar los conectores de entrada (Vac) y salida a la carga para que queden bien facil de conectar.
Parts:
- U1: symbol UC2844N -> UC2844N-RESCUE-PWM_JOSE_v1
Changed lines of the file:
@@
 EESchema Schematic File Version 2
+LIBS:PWM_JOSE_v1-rescue
 LIBS:power
 LIBS:device
@@
 $EndComp
 $Comp
-L UC2844N U1
+L UC2844N-RESCUE-PWM_JOSE_v1 U1
 U 1 1 5BD23F78
 P 3050 2050
