File: Kikad_PCBs/Placa_completa/Placa_completa.sch (KiCad schematic (older format))
At the start: 57 parts

Commit message: Placa final diseño completo.
Diseño kicad de la placa funcionando, falta hacer las modificaciones para que quede listo como para mandar a hacer, tambien modificar los conectores de entrada (Vac) y salida a la carga para que queden bien facil de conectar.
Parts:
- removed C? (x4): CP1, symbol CP1
- removed C? (x6): C, symbol C
- removed D?: D_Bridge_+AA-, symbol D_Bridge_+AA-
- removed D? (x3): D_Schottky, symbol D_Schottky
- removed D?: D, symbol D
- removed D? (x2): D_Zener, symbol D_Zener
- removed Q? (x2): Q_NPN_CBE, symbol Q_NPN_CBE
- removed R? (x16): R, symbol R
- removed T?: Transformer_1P_2S, symbol Transformer_1P_2S
- removed U?: UC2844N, DIP254P762X508-8, symbol UC2844N
- removed U?: TL431, TO-92, symbol TL431
- removed U?: PC817, Housings_DIP:DIP-4_W7.62mm, symbol PC817
- added D1: D_Bridge_-A+A, symbol D_Bridge_-A+A
- added D2: 20V, Diodes_THT:D_DO-41_SOD81_P7.62mm_Horizontal, symbol D_Zener
- added D4: Daux, Diodes_THT:D_DO-41_SOD81_P7.62mm_Horizontal, symbol D_Schottky
- added Dsec2: MUR860, TO_SOT_Packages_THT:TO-220-2_Vertical, symbol D
- added J1: Conn_01x03, Pin_Headers:Pin_Header_Straight_1x03_Pitch2.54mm, symbol Conn_01x03
- added J2: Vo+, Pin_Headers:Pin_Header_Straight_1x01_Pitch2.54mm, symbol Conn_01x01
- added J3: VoGnd, Pin_Headers:Pin_Header_Straight_1x01_Pitch2.54mm, symbol Conn_01x01
- added Rstartup1, Rstartup2: 75k, Resistors_THT:R_Axial_DIN0207_L6.3mm_D2.5mm_P7.62mm_Horizontal, symbol R
- added Rx1: 180k, Resistors_THT:R_Axial_DIN0309_L9.0mm_D3.2mm_P12.70mm_Horizontal, symbol R
- added T1: Transformer_1P_2S, Transformers_CHK:Trafo_CHK-EI30-2VA_1xSec, symbol Transformer_1P_2S
- added TH1: NTC, Capacitors_ThroughHole:C_Disc_D16.0mm_W5.0mm_P7.50mm, symbol Thermistor_NTC
- C1: renamed from C?; value C -> 1u; footprint (none) -> Capacitors_ThroughHole:C_Rect_L16.5mm_W5.0mm_P15.00mm_MKT
- C2: renamed from C?; value C -> 100n; footprint (none) -> Capacitors_THT:C_Rect_L7.0mm_W2.5mm_P5.00mm
- CBulk1: renamed from C?; value CP1 -> 220u; footprint (none) -> Capacitors_THT:CP_Axial_L42.0mm_D23.0mm_P45.00mm_Horizontal
- Cout1: renamed from C?; value C -> 380u; footprint (none) -> Capacitors_ThroughHole:CP_Radial_D22.0mm_P10.00mm_SnapIn
- Csnubb1: renamed from C?; value C -> 47n; footprint (none) -> Capacitors_THT:C_Disc_D5.0mm_W2.5mm_P2.50mm
- Cvcc1: renamed from C?; value CP1 -> 22u; footprint (none) -> Capacitors_THT:CP_Radial_D5.0mm_P2.00mm
- Cx1: renamed from C?; value CP1 -> 100n; footprint (none) -> Capacitors_THT:C_Rect_L16.5mm_W6.0mm_P15.00mm_MKT
- Cy1: renamed from C?; value C -> 100n; footprint (none) -> Capacitors_THT:C_Rect_L16.5mm_W6.0mm_P15.00mm_MKT
- Cy2: renamed from C?; value C -> 100N; footprint (none) -> Capacitors_THT:C_Rect_L16.5mm_W6.0mm_P15.00mm_MKT
- Dsec1: renamed from D?; value D -> MUR860; footprint (none) -> TO_SOT_Packages_THT:TO-220-2_Vertical
- Dsnub1: renamed from D?; footprint (none) -> TO_SOT_Packages_THT:TO-220-2_Vertical
- F1: renamed from F?; footprint (none) -> Fuse_Holders_and_Fuses:Fuseholder5x20_horiz_open_inline_Type-I
- FL1: renamed from FL?; value EMI_Filter_CommonMode -> EMI; footprint (none) -> Transformers_CHK:choke_tesis
- Q1: renamed from Q?; value Q_NMOS_GDS -> FQP5N60C; footprint (none) -> TO_SOT_Packages_THT:TO-220-3_Vertical
- Raux1: renamed from R?; value R -> 10k; footprint (none) -> Resistors_THT:R_Axial_DIN0309_L9.0mm_D3.2mm_P12.70mm_Horizontal
- Rsns1: renamed from R?; value R -> 0.33; footprint (none) -> Resistors_THT:R_Axial_DIN0309_L9.0mm_D3.2mm_P12.70mm_Horizontal
- Rsnubb1: renamed from R?; value R -> 6k8; footprint (none) -> Resistors_THT:R_Axial_DIN0411_L9.9mm_D3.6mm_P12.70mm_Horizontal
- Rsnubb2: renamed from R?; value R -> 6k8; footprint (none) -> Resistors_THT:R_Axial_DIN0309_L9.0mm_D3.2mm_P12.70mm_Horizontal
Connections:
- net labels added: Earth, GNDPWR
- net labels removed: Cbulk
- wire segments 149 -> 86
Other:
- moved on the sheet: C1, C2, CBulk1, Cout1, Csnubb1, Cvcc1, Cx1, Cy1, Cy2, Dsec1, Dsnub1, F1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

Commit message: Gant para presentar el 8/12 y modificaciones al PCB
Parts:
- removed J1: Conn_01x03, Pin_Headers:Pin_Header_Straight_1x03_Pitch2.54mm, symbol Conn_01x03
- added J1: L, Pin_Headers:Pin_Header_Straight_1x01_Pitch2.54mm, symbol Conn_01x01
- added J4: N, Pin_Headers:Pin_Header_Straight_1x01_Pitch2.54mm, symbol Conn_01x01
- added J5: Earth, Pin_Headers:Pin_Header_Straight_1x01_Pitch2.54mm, symbol Conn_01x01
- D1: footprint (none) -> Diodes_THT:Diode_Bridge_18.5x5.5
Connections:
- wire segments 86 -> 85
Changed lines of the file:
@@
-$EndComp
-$Comp
-L Conn_01x03 J1
-U 1 1 5C18A088
-P 2150 6150
-F 0 "J1" H 2150 6350 50  0000 C CNN
-F 1 "Conn_01x03" H 2150 5950 50  0000 C CNN
-F 2 "Pin_Headers:Pin_Header_Straight_1x03_Pitch2.54mm" H 2150 6150 50  0001 C CNN
-F 3 "" H 2150 6150 50  0001 C CNN
-	1    2150 6150
-	1    0    0    -1
 $EndComp
 $Comp
@@
 L Earth_Protective #PWR011
 U 1 1 5C18AAEE
-P 1700 6400
-F 0 "#PWR011" H 1950 6150 50  0001 C CNN
-F 1 "Earth_Protective" H 2150 6250 50  0001 C CNN
-F 2 "" H 1700 6300 50  0001 C CNN
-F 3 "" H 1700 6300 50  0001 C CNN
-	1    1700 6400
+P 1200 5850
+F 0 "#PWR011" H 1450 5600 50  0001 C CNN
+F 1 "Earth_Protective" H 1650 5700 50  0001 C CNN
+F 2 "" H 1200 5750 50  0001 C CNN
+F 3 "" H 1200 5750 50  0001 C CNN
+	1    1200 5850
 	1    0    0    -1
 $EndComp
@@
 L GNDPWR #PWR013
 U 1 1 5C18B250
-P 1350 6550
-F 0 "#PWR013" H 1350 6350 50  0001 C CNN
-F 1 "GNDPWR" H 1350 6420 50  0000 C CNN
-F 2 "" H 1350 6500 50  0001 C CNN
-F 3 "" H 1350 6500 50  0001 C CNN
-	1    1350 6550
+P 1200 5500
+F 0 "#PWR013" H 1200 5300 50  0001 C CNN
+F 1 "GNDPWR" H 1200 5370 50  0000 C CNN
+F 2 "" H 1200 5450 50  0001 C CNN
+F 3 "" H 1200 5450 50  0001 C CNN
+	1    1200 5500
 	1    0    0    -1
 $EndComp
@@
 L VAC #PWR014
 U 1 1 5C18B409
-P 1350 5900
-F 0 "#PWR014" H 1350 5800 50  0001 C CNN
-F 1 "VAC" H 1350 6150 50  0000 C CNN
-F 2 "" H 1350 5900 50  0001 C CNN
-F 3 "" H 1350 5900 50  0001 C CNN
-	1    1350 5900
+P 1200 4800
+F 0 "#PWR014" H 1200 4700 50  0001 C CNN
+F 1 "VAC" H 1200 5050 50  0000 C CNN
+F 2 "" H 1200 4800 50  0001 C CNN
+F 3 "" H 1200 4800 50  0001 C CNN
+	1    1200 4800
 	1    0    0    -1
 $EndComp
@@
 F 0 "D1" H 5000 2025 50  0000 L CNN
 F 1 "D_Bridge_-A+A" H 5000 1950 50  0000 L CNN
-F 2 "" H 4950 1750 50  0001 C CNN
+F 2 "Diodes_THT:Diode_Bridge_18.5x5.5" H 4950 1750 50  0001 C CNN
 F 3 "" H 4950 1750 50  0001 C CNN
 	1    4950 1750
@@
 	3500 5600 3500 5750
 Wire Wire Line
-	1950 6250 1700 6250
-Wire Wire Line
-	1700 6250 1700 6400
-Wire Wire Line
 	1200 2250 1200 2350
 Wire Wire Line
-	1950 6150 1350 6150
-Wire Wire Line
-	1350 6150 1350 6550
-Wire Wire Line
-	1350 5900 1350 6050
-Wire Wire Line
-	1350 6050 1950 6050
+	1800 5350 1200 5350
+Wire Wire Line
+	1200 4800 1200 4950
+Wire Wire Line
+	1200 4950 1800 4950
 Connection ~ 1200 1450
 Connection ~ 1200 2250
@@
 	1    0    0    -1
 $EndComp
+Wire Wire Line
+	1200 5350 1200 5500
+$Comp
+L Conn_01x01 J1
+U 1 1 5C548843
+P 2000 4950
+F 0 "J1" H 2000 5050 39  0000 C CNN
+F 1 "L" H 2000 4850 39  0000 C CNN
+F 2 "Pin_Headers:Pin_Header_Straight_1x01_Pitch2.54mm" H 2000 4950 50  0001 C CNN
+F 3 "" H 2000 4950 50  0001 C CNN
+	1    2000 4950
+	1    0    0    -1
+$EndComp
+$Comp
+L Conn_01x01 J4
+U 1 1 5C5488FB
+P 2000 5350
+F 0 "J4" H 2000 5450 39  0000 C CNN
+F 1 "N" H 2000 5250 39  0000 C CNN
+F 2 "Pin_Headers:Pin_Header_Straight_1x01_Pitch2.54mm" H 2000 5350 50  0001 C CNN
+F 3 "" H 2000 5350 50  0001 C CNN
+	1    2000 5350
+	1    0    0    -1
+$EndComp
+$Comp
+L Conn_01x01 J5
+U 1 1 5C54898A
+P 2000 5850
+F 0 "J5" H 2000 5950 39  0000 C CNN
+F 1 "Earth" H 2000 5750 39  0000 C CNN
+F 2 "Pin_Headers:Pin_Header_Straight_1x01_Pitch2.54mm" H 2000 5850 50  0001 C CNN
+F 3 "" H 2000 5850 50  0001 C CNN
+	1    2000 5850
+	1    0    0    -1
+$EndComp
+Wire Wire Line
+	1200 5850 1800 5850
 $EndSCHEMATC

Commit message: modificaciones al pcb
Parts:
- C1: value 1u -> 0.1u
- Cout1: value 380u -> 330u
- Csnubb1: value 47n -> 39p
- Cy2: value 100N -> 100n
- Daux1: renamed from D4; value Daux -> N1106; footprint Diodes_THT:D_DO-41_SOD81_P7.62mm_Horizontal -> TO_SOT_Packages_THT:TO-220-2_Vertical
- Dsec1, Dsec2: value MUR860 -> BYV29X
- Dsnub1: value D -> HER205
- NTC1: renamed from TH1; value NTC -> I5D20R
- Q1: value FQP5N60C -> FQP8N60C
- Raux1: value 10k -> 1k
- Rstartup1, Rstartup2: value 75k -> 82K
- renumbered D2 to DZ1
Changed lines of the file:
@@
 P 3550 2050
 F 0 "Cy2" H 3575 2150 39  0000 L CNN
-F 1 "100N" H 3575 1950 39  0000 L CNN
+F 1 "100n" H 3575 1950 39  0000 L CNN
 F 2 "Capacitors_THT:C_Rect_L16.5mm_W6.0mm_P15.00mm_MKT" H 3588 1900 50  0001 C CNN
 F 3 "" H 3550 2050 50  0001 C CNN
@@
 P 6400 1800
 F 0 "C1" H 6425 1900 50  0000 L CNN
-F 1 "1u" H 6425 1700 50  0000 L CNN
+F 1 "0.1u" H 6425 1700 50  0000 L CNN
 F 2 "Capacitors_ThroughHole:C_Rect_L16.5mm_W5.0mm_P15.00mm_MKT" H 6438 1650 50  0001 C CNN
 F 3 "" H 6400 1800 50  0001 C CNN
@@
 P 7700 1550
 F 0 "Csnubb1" H 7725 1650 50  0000 L CNN
-F 1 "47n" H 7725 1450 50  0000 L CNN
+F 1 "39p" H 7725 1450 50  0000 L CNN
 F 2 "Capacitors_THT:C_Disc_D5.0mm_W2.5mm_P2.50mm" H 7738 1400 50  0001 C CNN
 F 3 "" H 7700 1550 50  0001 C CNN
@@
 P 8050 1800
 F 0 "Dsnub1" H 8050 1900 50  0000 C CNN
-F 1 "D" H 8050 1700 50  0000 C CNN
+F 1 "HER205" H 8050 1700 50  0000 C CNN
 F 2 "TO_SOT_Packages_THT:TO-220-2_Vertical" H 8050 1800 50  0001 C CNN
 F 3 "" H 8050 1800 50  0001 C CNN
@@
 P 8200 3850
 F 0 "Q1" H 8400 3900 50  0000 L CNN
-F 1 "FQP5N60C" H 8400 3800 50  0000 L CNN
+F 1 "FQP8N60C" H 8400 3800 50  0000 L CNN
 F 2 "TO_SOT_Packages_THT:TO-220-3_Vertical" H 8400 3950 50  0001 C CNN
 F 3 "" H 8200 3850 50  0001 C CNN
@@
 P 8550 2550
 F 0 "Raux1" V 8630 2550 50  0000 C CNN
-F 1 "10k" V 8550 2550 39  0000 C CNN
+F 1 "1k" V 8550 2550 39  0000 C CNN
 F 2 "Resistors_THT:R_Axial_DIN0309_L9.0mm_D3.2mm_P12.70mm_Horizontal" V 8480 2550 50  0001 C CNN
 F 3 "" H 8550 2550 50  0001 C CNN
@@
 P 9900 1200
 F 0 "Dsec1" H 9900 1300 39  0000 C CNN
-F 1 "MUR860" H 9900 1100 39  0000 C CNN
+F 1 "BYV29X" H 9900 1100 39  0000 C CNN
 F 2 "TO_SOT_Packages_THT:TO-220-2_Vertical" H 9900 1200 50  0001 C CNN
 F 3 "" H 9900 1200 50  0001 C CNN
@@
 P 10550 1700
 F 0 "Cout1" H 10575 1800 50  0000 L CNN
-F 1 "380u" H 10575 1600 39  0000 L CNN
+F 1 "330u" H 10575 1600 39  0000 L CNN
 F 2 "Capacitors_ThroughHole:CP_Radial_D22.0mm_P10.00mm_SnapIn" H 10588 1550 50  0001 C CNN
 F 3 "" H 10550 1700 50  0001 C CNN
@@
 P 7000 1700
 F 0 "Rstartup1" V 7080 1700 39  0000 C CNN
-F 1 "75k" V 7000 1700 39  0000 C CNN
+F 1 "82K" V 7000 1700 39  0000 C CNN
 F 2 "Resistors_THT:R_Axial_DIN0207_L6.3mm_D2.5mm_P7.62mm_Horizontal" V 6930 1700 50  0001 C CNN
 F 3 "" H 7000 1700 50  0001 C CNN
@@
 P 7000 2250
 F 0 "Rstartup2" V 7080 2250 39  0000 C CNN
-F 1 "75k" V 7000 2250 39  0000 C CNN
+F 1 "82K" V 7000 2250 39  0000 C CNN
 F 2 "Resistors_THT:R_Axial_DIN0207_L6.3mm_D2.5mm_P7.62mm_Horizontal" V 6930 2250 50  0001 C CNN
 F 3 "" H 7000 2250 50  0001 C CNN
@@
 P 9900 1500
 F 0 "Dsec2" H 9900 1600 39  0000 C CNN
-F 1 "MUR860" H 9900 1400 39  0000 C CNN
+F 1 "BYV29X" H 9900 1400 39  0000 C CNN
 F 2 "TO_SOT_Packages_THT:TO-220-2_Vertical" H 9900 1500 50  0001 C CNN
 F 3 "" H 9900 1500 50  0001 C CNN
@@
 $EndComp
 $Comp
-L D_Zener D2
+L D_Zener DZ1
 U 1 1 5C1A5FEB
 P 8050 2850
-F 0 "D2" H 8050 2950 50  0000 C CNN
+F 0 "DZ1" H 8050 2950 50  0000 C CNN
 F 1 "20V" H 8050 2750 39  0000 C CNN
 F 2 "Diodes_THT:D_DO-41_SOD81_P7.62mm_Horizontal" H 8050 2850 50  0001 C CNN
@@
 $EndComp
 $Comp
-L Thermistor_NTC TH1
+L Thermistor_NTC NTC1
 U 1 1 5C1AC879
 P 4350 1450
-F 0 "TH1" V 4175 1450 39  0000 C CNN
-F 1 "NTC" V 4475 1450 39  0000 C CNN
+F 0 "NTC1" V 4175 1450 39  0000 C CNN
+F 1 "I5D20R" V 4475 1450 39  0000 C CNN
 F 2 "Capacitors_ThroughHole:C_Disc_D16.0mm_W5.0mm_P7.50mm" H 4350 1500 50  0001 C CNN
 F 3 "" H 4350 1500 50  0001 C CNN
@@
 $EndComp
 $Comp
-L D_Schottky D4
+L D_Schottky Daux1
 U 1 1 5C1AFBC9
 P 9000 2550
-F 0 "D4" H 9000 2650 39  0000 C CNN
-F 1 "Daux" H 9000 2450 39  0000 C CNN
-F 2 "Diodes_THT:D_DO-41_SOD81_P7.62mm_Horizontal" H 9000 2550 50  0001 C CNN
+F 0 "Daux1" H 9000 2650 39  0000 C CNN
+F 1 "N1106" H 9000 2450 39  0000 C CNN
+F 2 "TO_SOT_Packages_THT:TO-220-2_Vertical" H 9000 2550 50  0001 C CNN
 F 3 "" H 9000 2550 50  0001 C CNN
 	1    9000 2550
